File: HD-Driver.sch (KiCad schematic (older format))
At the start: 20 parts

Commit message: PCB's in progress
Parts:
- added C1: C, ~, symbol C
- added D1, D2: DIODE, ~, symbol DIODE
- added R1: R, ~, symbol R
- added RV1: POT, ~, symbol POT
- gave numbers to parts that had none: 20
Connections:
- wire segments 69 -> 80
Other:
- moved on the sheet: U1
