File: HD-Driver2.sch (KiCad schematic (older format))
At the start: 1 part

Commit message: PCB's in progress
Parts:
- gave numbers to parts that had none: 1
Changed lines of the file:
@@
 Sheet 2 2
 Title ""
-Date "12 mar 2014"
+Date "2 apr 2014"
 Rev ""
 Comp ""
@@
 $EndDescr
 $Comp
-L ATTINY85-P IC?
+L ATTINY85-P IC1
 U 1 1 531FA95C
 P 5050 3250
-F 0 "IC?" H 3900 3650 40  0000 C CNN
+F 0 "IC1" H 3900 3650 40  0000 C CNN
 F 1 "ATTINY85-P" H 6050 2850 40  0000 C CNN
 F 2 "DIP8" H 6050 3250 35  0000 C CIN
@@
 	3700 3200 3150 3200
 $Comp
-L GND #PWR?
+L GND #PWR018
 U 1 1 531FAC97
 P 6400 3700
-F 0 "#PWR?" H 6400 3700 30  0001 C CNN
+F 0 "#PWR018" H 6400 3700 30  0001 C CNN
 F 1 "GND" H 6400 3630 30  0001 C CNN
 F 2 "" H 6400 3700 60  0000 C CNN
@@
 $EndComp
 $Comp
-L +5V #PWR?
+L +5V #PWR019
 U 1 1 531FACD8
 P 6400 2700
-F 0 "#PWR?" H 6400 2790 20  0001 C CNN
+F 0 "#PWR019" H 6400 2790 20  0001 C CNN
 F 1 "+5V" H 6400 2790 30  0000 C CNN
 F 2 "" H 6400 2700 60  0000 C CNN
@@
 	3450 3000 3700 3000
 $Comp
-L +5V #PWR?
+L +5V #PWR020
 U 1 1 531FB264
 P 3450 2700
-F 0 "#PWR?" H 3450 2790 20  0001 C CNN
+F 0 "#PWR020" H 3450 2790 20  0001 C CNN
 F 1 "+5V" H 3450 2790 30  0000 C CNN
 F 2 "" H 3450 2700 60  0000 C CNN
